File: tiny13_light_switcher/Eagle/Attiny13/Attiny13.sch (EAGLE design)
At the start: 35 parts, among them J2 USB_A_PTH_MALE, Q4 2N7000, Q5 2N7000, Q6 2N7000, U1 ATTiny13, U2 ATTiny85

Commit message: Add pattern.
Parts:
- removed J2: USB_A_PTH_MALE, SparkFun-Connectors:USB_A_PTH_MALE
- added J1: USB_A_PTH_MALE, SparkFun-Connectors:USB_A_PTH_MALE
- added R7: R_LED16, MyLib:R0.125W_3P
- added R8: R_LED34, MyLib:R0.125W_3P
- added R9: R_LED25, MyLib:R0.125W_3P
- added USB1: USBA_RAW, MyParts:USBA_RAW
Connections:
- new net N$30: LED1.A, LED6.A, R7.2
- new net N$31: LED3.A, LED4.A, R8.2
- new net N$32: LED2.A, LED5.A, R9.2
- net AGND: now also J1.GND, USB1.GND; no longer J2.GND
- net N$1: now also J1.VBUS, USB1.VBUS; no longer J2.VBUS
- net N$19: now also J1.D+, USB1.D+; no longer J2.D+
- net N$4: now also J1.D-, USB1.D-; no longer J2.D-
- net VCC: now also R7.1, R8.1, R9.1; no longer LED1.A, LED2.A, LED3.A, LED4.A, LED5.A, LED6.A
Changed lines of the file:
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@@
 </variantdefs>
 <classes>
-<class number="0" name="default" width="0" drill="0">
+<class number="0" name="default" width="0.6096" drill="0">
+<clearance class="0" value="0.508"/>
+</class>
+<class number="1" name="Power" width="0.9144" drill="0">
+<clearance class="1" value="0.9144"/>
 </class>
 </classes>
@@
 <part name="SUPPLY17" library="supply2" library_urn="urn:adsk.eagle:library:372" deviceset="AGND" device=""/>
 <part name="SUPPLY18" library="supply2" library_urn="urn:adsk.eagle:library:372" deviceset="AGND" device=""/>
-<part name="J2" library="SparkFun-Connectors" deviceset="USB_A" device="_PTH_MALE"/>
+<part name="J1" library="SparkFun-Connectors" deviceset="USB_A" device="_PTH_MALE"/>
+<part name="USB1" library="MyParts" deviceset="USBA_RAW" device=""/>
+<part name="R7" library="MyLib" deviceset="R" device="0.125W_3P" value="R_LED16"/>
+<part name="R8" library="MyLib" deviceset="R" device="0.125W_3P" value="R_LED34"/>
+<part name="R9" library="MyLib" deviceset="R" device="0.125W_3P" value="R_LED25"/>
 </parts>
 <sheets>
@@
 <instance part="SUPPLY17" gate="G$1" x="38.1" y="53.34" rot="R270"/>
 <instance part="SUPPLY18" gate="G$1" x="101.6" y="50.8"/>
-<instance part="J2" gate="G$1" x="53.34" y="152.4" rot="R90"/>
+<instance part="J1" gate="G$1" x="50.8" y="162.56" rot="R90"/>
+<instance part="USB1" gate="G$1" x="73.66" y="162.56" rot="R270"/>
+<instance part="R7" gate="G$1" x="149.86" y="96.52" rot="R270"/>
+<instance part="R8" gate="G$1" x="187.96" y="96.52" rot="R270"/>
+<instance part="R9" gate="G$1" x="231.14" y="96.52" rot="R270"/>
 </instances>
 <busses>
 </busses>
 <nets>
-<net name="GND" class="0">
+<net name="GND" class="1">
 <segment>
 <pinref part="C5" gate="G$1" pin="1"/>
@@
 </segment>
 </net>
-<net name="VCC" class="0">
+<net name="VCC" class="1">
 <segment>
 <wire x1="124.46" y1="154.94" x2="124.46" y2="149.86" width="0.1524" layer="91"/>
@@
 <pinref part="VCC4" gate="VCC" pin="VCC"/>
 <wire x1="119.38" y1="104.14" x2="149.86" y2="104.14" width="0.1524" layer="91"/>
-<pinref part="LED1" gate="G$1" pin="A"/>
-<wire x1="149.86" y1="104.14" x2="149.86" y2="88.9" width="0.1524" layer="91"/>
-<wire x1="149.86" y1="104.14" x2="160.02" y2="104.14" width="0.1524" layer="91"/>
+<pinref part="R7" gate="G$1" pin="1"/>
+<wire x1="149.86" y1="104.14" x2="187.96" y2="104.14" width="0.1524" layer="91"/>
+<wire x1="187.96" y1="104.14" x2="231.14" y2="104.14" width="0.1524" layer="91"/>
+<wire x1="149.86" y1="101.6" x2="149.86" y2="104.14" width="0.1524" layer="91"/>
 <junction x="149.86" y="104.14"/>
-<pinref part="LED6" gate="G$1" pin="A"/>
-<wire x1="160.02" y1="104.14" x2="160.02" y2="88.9" width="0.1524" layer="91"/>
-<wire x1="160.02" y1="104.14" x2="187.96" y2="104.14" width="0.1524" layer="91"/>
-<junction x="160.02" y="104.14"/>
-<pinref part="LED4" gate="G$1" pin="A"/>
-<wire x1="187.96" y1="104.14" x2="187.96" y2="88.9" width="0.1524" layer="91"/>
-<wire x1="187.96" y1="104.14" x2="198.12" y2="104.14" width="0.1524" layer="91"/>
+<pinref part="R8" gate="G$1" pin="1"/>
+<wire x1="187.96" y1="101.6" x2="187.96" y2="104.14" width="0.1524" layer="91"/>
 <junction x="187.96" y="104.14"/>
-<pinref part="LED3" gate="G$1" pin="A"/>
-<wire x1="198.12" y1="104.14" x2="198.12" y2="88.9" width="0.1524" layer="91"/>
-<wire x1="198.12" y1="104.14" x2="231.14" y2="104.14" width="0.1524" layer="91"/>
-<junction x="198.12" y="104.14"/>
-<pinref part="LED5" gate="G$1" pin="A"/>
-<wire x1="231.14" y1="104.14" x2="231.14" y2="88.9" width="0.1524" layer="91"/>
-<wire x1="231.14" y1="104.14" x2="241.3" y2="104.14" width="0.1524" layer="91"/>
-<junction x="231.14" y="104.14"/>
-<pinref part="LED2" gate="G$1" pin="A"/>
-<wire x1="241.3" y1="104.14" x2="241.3" y2="88.9" width="0.1524" layer="91"/>
+<pinref part="R9" gate="G$1" pin="1"/>
+<wire x1="231.14" y1="101.6" x2="231.14" y2="104.14" width="0.1524" layer="91"/>
 </segment>
 </net>
@@
 </segment>
 </net>
-<net name="N$1" class="0">
+<net name="N$1" class="1">
 <segment>
 <pinref part="D1" gate="G$1" pin="C"/>
-<wire x1="33.02" y1="137.16" x2="48.26" y2="137.16" width="0.1524" layer="91"/>
-<wire x1="48.26" y1="137.16" x2="48.26" y2="144.78" width="0.1524" layer="91"/>
-<pinref part="J2" gate="G$1" pin="VBUS"/>
+<wire x1="33.02" y1="137.16" x2="45.72" y2="137.16" width="0.1524" layer="91"/>
+<wire x1="45.72" y1="137.16" x2="45.72" y2="154.94" width="0.1524" layer="91"/>
+<pinref part="J1" gate="G$1" pin="VBUS"/>
+<wire x1="45.72" y1="154.94" x2="45.72" y2="165.1" width="0.1524" layer="91"/>
+<junction x="45.72" y="154.94"/>
+<wire x1="45.72" y1="165.1" x2="76.2" y2="165.1" width="0.1524" layer="91"/>
+<wire x1="76.2" y1="165.1" x2="76.2" y2="152.4" width="0.1524" layer="91"/>
+<pinref part="USB1" gate="G$1" pin="VBUS"/>
 </segment>
 </net>
 <net name="N$4" class="0">
 <segment>
-<wire x1="50.8" y1="129.54" x2="50.8" y2="144.78" width="0.1524" layer="91"/>
 <pinref part="D2" gate="G$1" pin="C"/>
 <wire x1="50.8" y1="129.54" x2="60.96" y2="129.54" width="0.1524" layer="91"/>
@@
 <wire x1="50.8" y1="109.22" x2="50.8" y2="124.46" width="0.1524" layer="91"/>
 <junction x="50.8" y="124.46"/>
-<pinref part="J2" gate="G$1" pin="D-"/>
+<wire x1="50.8" y1="129.54" x2="50.8" y2="142.24" width="0.1524" layer="91"/>
+<wire x1="50.8" y1="142.24" x2="48.26" y2="142.24" width="0.1524" layer="91"/>
+<pinref part="J1" gate="G$1" pin="D-"/>
+<wire x1="48.26" y1="142.24" x2="48.26" y2="154.94" width="0.1524" layer="91"/>
+<wire x1="48.26" y1="154.94" x2="48.26" y2="162.56" width="0.1524" layer="91"/>
+<junction x="48.26" y="154.94"/>
+<wire x1="48.26" y1="162.56" x2="71.12" y2="162.56" width="0.1524" layer="91"/>
+<wire x1="71.12" y1="162.56" x2="71.12" y2="152.4" width="0.1524" layer="91"/>
+<pinref part="USB1" gate="G$1" pin="D-"/>
 </segment>
 </net>
@@
 <segment>
 <pinref part="D3" gate="G$1" pin="C"/>
-<wire x1="53.34" y1="144.78" x2="53.34" y2="137.16" width="0.1524" layer="91"/>
 <wire x1="53.34" y1="137.16" x2="60.96" y2="137.16" width="0.1524" layer="91"/>
 <junction x="53.34" y="137.16"/>
@@
 <wire x1="53.34" y1="116.84" x2="45.72" y2="116.84" width="0.1524" layer="91"/>
 <pinref part="R1" gate="G$1" pin="2"/>
-<pinref part="J2" gate="G$1" pin="D+"/>
+<wire x1="53.34" y1="137.16" x2="53.34" y2="147.32" width="0.1524" layer="91"/>
+<pinref part="J1" gate="G$1" pin="D+"/>
+<wire x1="53.34" y1="147.32" x2="50.8" y2="147.32" width="0.1524" layer="91"/>
+<wire x1="50.8" y1="147.32" x2="50.8" y2="154.94" width="0.1524" layer="91"/>
+<wire x1="50.8" y1="154.94" x2="50.8" y2="160.02" width="0.1524" layer="91"/>
+<junction x="50.8" y="154.94"/>
+<wire x1="50.8" y1="160.02" x2="73.66" y2="160.02" width="0.1524" layer="91"/>
+<wire x1="73.66" y1="160.02" x2="73.66" y2="152.4" width="0.1524" layer="91"/>
+<pinref part="USB1" gate="G$1" pin="D+"/>
 </segment>
 </net>
@@
 </segment>
 </net>
-<net name="AGND" class="0">
+<net name="AGND" class="1">
 <segment>
 <pinref part="C1" gate="G$1" pin="1"/>
@@
 </segment>
 <segment>
-<wire x1="55.88" y1="144.78" x2="68.58" y2="144.78" width="0.1524" layer="91"/>
 <pinref part="SUPPLY13" gate="G$1" pin="AGND"/>
-<pinref part="J2" gate="G$1" pin="GND"/>
+<wire x1="68.58" y1="144.78" x2="55.88" y2="144.78" width="0.1524" layer="91"/>
+<wire x1="55.88" y1="144.78" x2="55.88" y2="149.86" width="0.1524" layer="91"/>
+<wire x1="55.88" y1="149.86" x2="53.34" y2="149.86" width="0.1524" layer="91"/>
+<pinref part="J1" gate="G$1" pin="GND"/>
+<wire x1="53.34" y1="149.86" x2="53.34" y2="154.94" width="0.1524" layer="91"/>
+<wire x1="53.34" y1="154.94" x2="63.5" y2="154.94" width="0.1524" layer="91"/>
+<wire x1="63.5" y1="154.94" x2="63.5" y2="152.4" width="0.1524" layer="91"/>
+<junction x="53.34" y="154.94"/>
+<wire x1="63.5" y1="152.4" x2="68.58" y2="152.4" width="0.1524" layer="91"/>
+<pinref part="USB1" gate="G$1" pin="GND"/>
 </segment>
 <segment>
@@
 </segment>
 </net>
+<net name="N$30" class="0">
+<segment>
+<pinref part="R7" gate="G$1" pin="2"/>
+<pinref part="LED1" gate="G$1" pin="A"/>
+<wire x1="149.86" y1="91.44" x2="149.86" y2="88.9" width="0.1524" layer="91"/>
+<wire x1="149.86" y1="91.44" x2="160.02" y2="91.44" width="0.1524" layer="91"/>
+<junction x="149.86" y="91.44"/>
+<pinref part="LED6" gate="G$1" pin="A"/>
+<wire x1="160.02" y1="91.44" x2="160.02" y2="88.9" width="0.1524" layer="91"/>
+</segment>
+</net>
+<net name="N$31" class="0">
+<segment>
+<pinref part="R8" gate="G$1" pin="2"/>
+<pinref part="LED4" gate="G$1" pin="A"/>
+<wire x1="187.96" y1="91.44" x2="187.96" y2="88.9" width="0.1524" layer="91"/>
+<wire x1="187.96" y1="91.44" x2="198.12" y2="91.44" width="0.1524" layer="91"/>
+<junction x="187.96" y="91.44"/>
+<pinref part="LED3" gate="G$1" pin="A"/>
+<wire x1="198.12" y1="91.44" x2="198.12" y2="88.9" width="0.1524" layer="91"/>
+</segment>
+</net>
+<net name="N$32" class="0">
+<segment>
+<pinref part="LED5" gate="G$1" pin="A"/>
+<pinref part="R9" gate="G$1" pin="2"/>
+<wire x1="231.14" y1="88.9" x2="231.14" y2="91.44" width="0.1524" layer="91"/>
+<wire x1="231.14" y1="91.44" x2="241.3" y2="91.44" width="0.1524" layer="91"/>
+<junction x="231.14" y="91.44"/>
+<pinref part="LED2" gate="G$1" pin="A"/>
+<wire x1="241.3" y1="91.44" x2="241.3" y2="88.9" width="0.1524" layer="91"/>
+</segment>
+</net>

Commit message: Fix USB & parts layout.
Parts:
- removed J1: USB_A_PTH_MALE, SparkFun-Connectors:USB_A_PTH_MALE
- added U$2: USB_MY_BREAKOUT, MyParts:USB_MY_BREAKOUT
Connections:
- net AGND: now also U$2.GND; no longer J1.GND
- net N$1: now also U$2.VBUS; no longer J1.VBUS
- net N$19: now also U$2.D+; no longer J1.D+
- net N$4: now also U$2.D-; no longer J1.D-
Changed lines of the file:
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@@
 <part name="SUPPLY17" library="supply2" library_urn="urn:adsk.eagle:library:372" deviceset="AGND" device=""/>
 <part name="SUPPLY18" library="supply2" library_urn="urn:adsk.eagle:library:372" deviceset="AGND" device=""/>
-<part name="J1" library="SparkFun-Connectors" deviceset="USB_A" device="_PTH_MALE"/>
-<part name="USB1" library="MyParts" deviceset="USBA_RAW" device=""/>
 <part name="R7" library="MyLib" deviceset="R" device="0.125W_3P" value="R_LED16"/>
 <part name="R8" library="MyLib" deviceset="R" device="0.125W_3P" value="R_LED34"/>
 <part name="R9" library="MyLib" deviceset="R" device="0.125W_3P" value="R_LED25"/>
+<part name="U$2" library="MyParts" deviceset="USB_MY_BREAKOUT" device=""/>
+<part name="USB1" library="MyParts" deviceset="USBA_RAW" device=""/>
 </parts>
 <sheets>
@@
 <instance part="SUPPLY17" gate="G$1" x="38.1" y="53.34" rot="R270"/>
 <instance part="SUPPLY18" gate="G$1" x="101.6" y="50.8"/>
-<instance part="J1" gate="G$1" x="50.8" y="162.56" rot="R90"/>
-<instance part="USB1" gate="G$1" x="73.66" y="162.56" rot="R270"/>
 <instance part="R7" gate="G$1" x="149.86" y="96.52" rot="R270"/>
 <instance part="R8" gate="G$1" x="187.96" y="96.52" rot="R270"/>
 <instance part="R9" gate="G$1" x="231.14" y="96.52" rot="R270"/>
+<instance part="U$2" gate="G$1" x="48.26" y="165.1" rot="R90"/>
+<instance part="USB1" gate="G$1" x="73.66" y="162.56" rot="R270"/>
 </instances>
 <busses>
@@
 </segment>
 </net>
-<net name="+5V" class="0">
+<net name="+5V" class="1">
 <segment>
 <pinref part="U2" gate="G$1" pin="VCC"/>
@@
 <wire x1="33.02" y1="137.16" x2="45.72" y2="137.16" width="0.1524" layer="91"/>
 <wire x1="45.72" y1="137.16" x2="45.72" y2="154.94" width="0.1524" layer="91"/>
-<pinref part="J1" gate="G$1" pin="VBUS"/>
 <wire x1="45.72" y1="154.94" x2="45.72" y2="165.1" width="0.1524" layer="91"/>
-<junction x="45.72" y="154.94"/>
 <wire x1="45.72" y1="165.1" x2="76.2" y2="165.1" width="0.1524" layer="91"/>
 <wire x1="76.2" y1="165.1" x2="76.2" y2="152.4" width="0.1524" layer="91"/>
+<pinref part="U$2" gate="G$1" pin="VBUS"/>
+<junction x="45.72" y="154.94"/>
 <pinref part="USB1" gate="G$1" pin="VBUS"/>
 </segment>
@@
 <wire x1="50.8" y1="129.54" x2="50.8" y2="142.24" width="0.1524" layer="91"/>
 <wire x1="50.8" y1="142.24" x2="48.26" y2="142.24" width="0.1524" layer="91"/>
-<pinref part="J1" gate="G$1" pin="D-"/>
 <wire x1="48.26" y1="142.24" x2="48.26" y2="154.94" width="0.1524" layer="91"/>
 <wire x1="48.26" y1="154.94" x2="48.26" y2="162.56" width="0.1524" layer="91"/>
-<junction x="48.26" y="154.94"/>
 <wire x1="48.26" y1="162.56" x2="71.12" y2="162.56" width="0.1524" layer="91"/>
 <wire x1="71.12" y1="162.56" x2="71.12" y2="152.4" width="0.1524" layer="91"/>
+<pinref part="U$2" gate="G$1" pin="D-"/>
+<junction x="48.26" y="154.94"/>
 <pinref part="USB1" gate="G$1" pin="D-"/>
 </segment>
@@
 <pinref part="R1" gate="G$1" pin="2"/>
 <wire x1="53.34" y1="137.16" x2="53.34" y2="147.32" width="0.1524" layer="91"/>
-<pinref part="J1" gate="G$1" pin="D+"/>
 <wire x1="53.34" y1="147.32" x2="50.8" y2="147.32" width="0.1524" layer="91"/>
 <wire x1="50.8" y1="147.32" x2="50.8" y2="154.94" width="0.1524" layer="91"/>
 <wire x1="50.8" y1="154.94" x2="50.8" y2="160.02" width="0.1524" layer="91"/>
-<junction x="50.8" y="154.94"/>
 <wire x1="50.8" y1="160.02" x2="73.66" y2="160.02" width="0.1524" layer="91"/>
 <wire x1="73.66" y1="160.02" x2="73.66" y2="152.4" width="0.1524" layer="91"/>
+<pinref part="U$2" gate="G$1" pin="D+"/>
+<junction x="50.8" y="154.94"/>
 <pinref part="USB1" gate="G$1" pin="D+"/>
 </segment>
@@
 <wire x1="55.88" y1="144.78" x2="55.88" y2="149.86" width="0.1524" layer="91"/>
 <wire x1="55.88" y1="149.86" x2="53.34" y2="149.86" width="0.1524" layer="91"/>
-<pinref part="J1" gate="G$1" pin="GND"/>
 <wire x1="53.34" y1="149.86" x2="53.34" y2="154.94" width="0.1524" layer="91"/>
 <wire x1="53.34" y1="154.94" x2="63.5" y2="154.94" width="0.1524" layer="91"/>
 <wire x1="63.5" y1="154.94" x2="63.5" y2="152.4" width="0.1524" layer="91"/>
+<wire x1="63.5" y1="152.4" x2="68.58" y2="152.4" width="0.1524" layer="91"/>
+<pinref part="U$2" gate="G$1" pin="GND"/>
 <junction x="53.34" y="154.94"/>
-<wire x1="63.5" y1="152.4" x2="68.58" y2="152.4" width="0.1524" layer="91"/>
 <pinref part="USB1" gate="G$1" pin="GND"/>
 </segment>

Commit message: Change capacitor package.
Parts:
- C1, C2: device MyLib:CAPDIP_1 -> MyLib:CAPDIP_2
Changed lines of the file:
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@@
 <grid distance="0.1" unitdist="inch" unit="inch" style="lines" multiple="1" display="no" altdistance="0.01" altunitdist="inch" altunit="inch"/>
 <layers>
-<layer number="1" name="Top" color="4" fill="1" visible="no" active="no"/>
-<layer number="16" name="Bottom" color="1" fill="1" visible="no" active="no"/>
-<layer number="17" name="Pads" color="2" fill="1" visible="no" active="no"/>
-<layer number="18" name="Vias" color="2" fill="1" visible="no" active="no"/>
-<layer number="19" name="Unrouted" color="6" fill="1" visible="no" active="no"/>
-<layer number="20" name="Dimension" color="15" fill="1" visible="no" active="no"/>
-<layer number="21" name="tPlace" color="7" fill="1" visible="no" active="no"/>
-<layer number="22" name="bPlace" color="7" fill="1" visible="no" active="no"/>
-<layer number="23" name="tOrigins" color="15" fill="1" visible="no" active="no"/>
-<layer number="24" name="bOrigins" color="15" fill="1" visible="no" active="no"/>
-<layer number="25" name="tNames" color="7" fill="1" visible="no" active="no"/>
-<layer number="26" name="bNames" color="7" fill="1" visible="no" active="no"/>
-<layer number="27" name="tValues" color="7" fill="1" visible="no" active="no"/>
-<layer number="28" name="bValues" color="7" fill="1" visible="no" active="no"/>
+<layer number="1" name="Top" color="4" fill="1" visible="yes" active="no"/>
+<layer number="16" name="Bottom" color="1" fill="1" visible="yes" active="no"/>
+<layer number="17" name="Pads" color="2" fill="1" visible="yes" active="no"/>
+<layer number="18" name="Vias" color="2" fill="1" visible="yes" active="no"/>
+<layer number="19" name="Unrouted" color="6" fill="1" visible="yes" active="no"/>
+<layer number="20" name="Dimension" color="15" fill="1" visible="yes" active="no"/>
+<layer number="21" name="tPlace" color="7" fill="1" visible="yes" active="no"/>
+<layer number="22" name="bPlace" color="7" fill="1" visible="yes" active="no"/>
+<layer number="23" name="tOrigins" color="15" fill="1" visible="yes" active="no"/>
+<layer number="24" name="bOrigins" color="15" fill="1" visible="yes" active="no"/>
+<layer number="25" name="tNames" color="7" fill="1" visible="yes" active="no"/>
+<layer number="26" name="bNames" color="7" fill="1" visible="yes" active="no"/>
+<layer number="27" name="tValues" color="7" fill="1" visible="yes" active="no"/>
+<layer number="28" name="bValues" color="7" fill="1" visible="yes" active="no"/>
 <layer number="29" name="tStop" color="7" fill="3" visible="no" active="no"/>
 <layer number="30" name="bStop" color="7" fill="6" visible="no" active="no"/>
@@
 <layer number="35" name="tGlue" color="7" fill="4" visible="no" active="no"/>
 <layer number="36" name="bGlue" color="7" fill="5" visible="no" active="no"/>
-<layer number="37" name="tTest" color="7" fill="1" visible="no" active="no"/>
-<layer number="38" name="bTest" color="7" fill="1" visible="no" active="no"/>
+<layer number="37" name="tTest" color="7" fill="1" visible="yes" active="no"/>
+<layer number="38" name="bTest" color="7" fill="1" visible="yes" active="no"/>
 <layer number="39" name="tKeepout" color="4" fill="11" visible="no" active="no"/>
 <layer number="40" name="bKeepout" color="1" fill="11" visible="no" active="no"/>
@@
 <layer number="44" name="Drills" color="7" fill="1" visible="no" active="no"/>
 <layer number="45" name="Holes" color="7" fill="1" visible="no" active="no"/>
-<layer number="46" name="Milling" color="3" fill="1" visible="no" active="no"/>
-<layer number="47" name="Measures" color="7" fill="1" visible="no" active="no"/>
-<layer number="48" name="Document" color="7" fill="1" visible="no" active="no"/>
-<layer number="49" name="Reference" color="7" fill="1" visible="no" active="no"/>
-<layer number="50" name="dxf" color="7" fill="1" visible="no" active="no"/>
-<layer number="51" name="tDocu" color="7" fill="1" visible="no" active="no"/>
-<layer number="52" name="bDocu" color="7" fill="1" visible="no" active="no"/>
-<layer number="53" name="tGND_GNDA" color="7" fill="1" visible="no" active="no"/>
-<layer number="54" name="bGND_GNDA" color="7" fill="1" visible="no" active="no"/>
-<layer number="56" name="wert" color="7" fill="1" visible="no" active="no"/>
-<layer number="57" name="tCAD" color="7" fill="1" visible="no" active="no"/>
-<layer number="59" name="tCarbon" color="7" fill="1" visible="no" active="no"/>
-<layer number="60" name="bCarbon" color="7" fill="1" visible="no" active="no"/>
+<layer number="46" name="Milling" color="3" fill="1" visible="yes" active="no"/>
+<layer number="47" name="Measures" color="7" fill="1" visible="yes" active="no"/>
+<layer number="48" name="Document" color="7" fill="1" visible="yes" active="no"/>
+<layer number="49" name="Reference" color="7" fill="1" visible="yes" active="no"/>
+<layer number="50" name="dxf" color="7" fill="1" visible="yes" active="no"/>
+<layer number="51" name="tDocu" color="7" fill="1" visible="yes" active="no"/>
+<layer number="52" name="bDocu" color="7" fill="1" visible="yes" active="no"/>
+<layer number="53" name="tGND_GNDA" color="7" fill="1" visible="yes" active="no"/>
+<layer number="54" name="bGND_GNDA" color="7" fill="1" visible="yes" active="no"/>
+<layer number="56" name="wert" color="7" fill="1" visible="yes" active="no"/>
+<layer number="57" name="tCAD" color="7" fill="1" visible="yes" active="no"/>
+<layer number="59" name="tCarbon" color="7" fill="1" visible="yes" active="no"/>
+<layer number="60" name="bCarbon" color="7" fill="1" visible="yes" active="no"/>
 <layer number="90" name="Modules" color="5" fill="1" visible="yes" active="yes"/>
 <layer number="91" name="Nets" color="2" fill="1" visible="yes" active="yes"/>
@@
 <clearance class="0" value="0.508"/>
 </class>
-<class number="1" name="Power" width="0.9144" drill="0">
-<clearance class="1" value="0.9144"/>
+<class number="1" name="Power" width="0.762" drill="0">
+<clearance class="1" value="0.762"/>
 </class>
 </classes>
@@
 <part name="ESDV_R" library="adafruit" deviceset="PINHD-1X10" device=""/>
 <part name="ESDV_L" library="adafruit" deviceset="PINHD-1X10" device=""/>
-<part name="C2" library="MyLib" deviceset="CAP" device="DIP_1" value="4.7uF"/>
+<part name="C2" library="MyLib" deviceset="CAP" device="DIP_2" value="4.7uF"/>
 <part name="P+5" library="supply1" library_urn="urn:adsk.eagle:library:371" deviceset="+5V" device=""/>
-<part name="C1" library="MyLib" deviceset="CAP" device="DIP_1" value="0.1uF"/>
+<part name="C1" library="MyLib" deviceset="CAP" device="DIP_2" value="0.1uF"/>
 <part name="SUPPLY9" library="supply2" library_urn="urn:adsk.eagle:library:372" deviceset="VDD" device=""/>
 <part name="JP3" library="pinhead" library_urn="urn:adsk.eagle:library:325" deviceset="PINHD-1X3" device="" value="VINSEL"/>
